File: macropad/macropad-rev1/macropad-rev1.kicad_sch (KiCad schematic)
At the start: 30 parts, among them Q1 2N7000, Q2 2N7000, Q3 2N7000, Q4 2N7000, SW10 RotaryEncoder_Switch, U1 Pico, U2 MDOB128032GV-WI

Commit message: Now using SVG and drill marks
Parts:
- SW1, SW2, SW3, SW4, SW5, SW6, SW7, SW8, SW9: footprint LiveWires:LW_CherrySwitch -> LiveWires:LW_CherrySwitch_DrillMarks
Changed lines of the file:
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@@
 		)
 		(instances
-			(project "macroboard-rev1"
+			(project "macropad-rev1"
 				(path "/e2f35591-d2a5-4370-be80-1eddbbb1c064"
 					(reference "#PWR010")
@@
 		)
 		(instances
-			(project "macroboard-rev1"
+			(project "macropad-rev1"
 				(path "/e2f35591-d2a5-4370-be80-1eddbbb1c064"
 					(reference "#PWR02")
@@
 		)
 		(instances
-			(project "macroboard-rev1"
+			(project "macropad-rev1"
 				(path "/e2f35591-d2a5-4370-be80-1eddbbb1c064"
 					(reference "#PWR05")
@@
 			)
 		)
-		(property "Footprint" "LiveWires:LW_CherrySwitch"
+		(property "Footprint" "LiveWires:LW_CherrySwitch_DrillMarks"
 			(at 52.07 62.23 0)
 			(effects
@@
 		)
 		(instances
-			(project "macroboard-rev1"
+			(project "macropad-rev1"
 				(path "/e2f35591-d2a5-4370-be80-1eddbbb1c064"
 					(reference "SW9")
@@
 		)
 		(instances
-			(project "macroboard-rev1"
+			(project "macropad-rev1"
 				(path "/e2f35591-d2a5-4370-be80-1eddbbb1c064"
 					(reference "D4")
@@
 			)
 		)
-		(property "Footprint" "LiveWires:LW_CherrySwitch"
+		(property "Footprint" "LiveWires:LW_CherrySwitch_DrillMarks"
 			(at 199.39 115.57 0)
 			(effects
@@
 		)
 		(instances
-			(project "macroboard-rev1"
+			(project "macropad-rev1"
 				(path "/e2f35591-d2a5-4370-be80-1eddbbb1c064"
 					(reference "SW5")
@@
 		)
 		(instances
-			(project "macroboard-rev1"
+			(project "macropad-rev1"
 				(path "/e2f35591-d2a5-4370-be80-1eddbbb1c064"
 					(reference "C1")
@@
 		)
 		(instances
-			(project "macroboard-rev1"
+			(project "macropad-rev1"
 				(path "/e2f35591-d2a5-4370-be80-1eddbbb1c064"
 					(reference "#PWR015")
@@
 		)
 		(instances
-			(project "macroboard-rev1"
+			(project "macropad-rev1"
 				(path "/e2f35591-d2a5-4370-be80-1eddbbb1c064"
 					(reference "Q2")
@@
 		)
 		(instances
-			(project "macroboard-rev1"
+			(project "macropad-rev1"
 				(path "/e2f35591-d2a5-4370-be80-1eddbbb1c064"
 					(reference "D1")
@@
 		)
 		(instances
-			(project "macroboard-rev1"
+			(project "macropad-rev1"
 				(path "/e2f35591-d2a5-4370-be80-1eddbbb1c064"
 					(reference "C2")
@@
 		)
 		(instances
-			(project "macroboard-rev1"
+			(project "macropad-rev1"
 				(path "/e2f35591-d2a5-4370-be80-1eddbbb1c064"
 					(reference "R8")
@@
 		)
 		(instances
-			(project "macroboard-rev1"
+			(project "macropad-rev1"
 				(path "/e2f35591-d2a5-4370-be80-1eddbbb1c064"
 					(reference "D2")
@@
 		)
 		(instances
-			(project "macroboard-rev1"
+			(project "macropad-rev1"
 				(path "/e2f35591-d2a5-4370-be80-1eddbbb1c064"
 					(reference "#PWR017")
@@
 		)
 		(instances
-			(project "macroboard-rev1"
+			(project "macropad-rev1"
 				(path "/e2f35591-d2a5-4370-be80-1eddbbb1c064"
 					(reference "#PWR04")
@@
 			)
 		)
-		(property "Footprint" "LiveWires:LW_CherrySwitch"
+		(property "Footprint" "LiveWires:LW_CherrySwitch_DrillMarks"
 			(at 52.07 90.17 0)
 			(effects
@@
 		)
 		(instances
-			(project "macroboard-rev1"
+			(project "macropad-rev1"
 				(path "/e2f35591-d2a5-4370-be80-1eddbbb1c064"
 					(reference "SW3")
@@
 			)
 		)
-		(property "Footprint" "LiveWires:LW_CherrySwitch"
+		(property "Footprint" "LiveWires:LW_CherrySwitch_DrillMarks"
 			(at 52.07 82.55 0)
 			(effects
@@
 		)
 		(instances
-			(project "macroboard-rev1"
+			(project "macropad-rev1"
 				(path "/e2f35591-d2a5-4370-be80-1eddbbb1c064"
 					(reference "SW2")
@@
 		)
 		(instances
-			(project "macroboard-rev1"
+			(project "macropad-rev1"
 				(path "/e2f35591-d2a5-4370-be80-1eddbbb1c064"
 					(reference "Q3")
@@
 			)
 		)
-		(property "Footprint" "LiveWires:LW_CherrySwitch"
+		(property "Footprint" "LiveWires:LW_CherrySwitch_DrillMarks"
 			(at 199.39 138.43 0)
 			(effects
@@
 		)
 		(instances
-			(project "macroboard-rev1"
+			(project "macropad-rev1"
 				(path "/e2f35591-d2a5-4370-be80-1eddbbb1c064"
 					(reference "SW8")
@@
 		)
 		(instances
-			(project "macroboard-rev1"
+			(project "macropad-rev1"
 				(path "/e2f35591-d2a5-4370-be80-1eddbbb1c064"
 					(reference "#PWR06")
@@
 		)
 		(instances
-			(project "macroboard-rev1"
+			(project "macropad-rev1"
 				(path "/e2f35591-d2a5-4370-be80-1eddbbb1c064"
 					(reference "U2")
@@
 		)
 		(instances
-			(project "macroboard-rev1"
+			(project "macropad-rev1"
 				(path "/e2f35591-d2a5-4370-be80-1eddbbb1c064"
 					(reference "Q1")
@@
 		)
 		(instances
-			(project "macroboard-rev1"
+			(project "macropad-rev1"
 				(path "/e2f35591-d2a5-4370-be80-1eddbbb1c064"
 					(reference "#PWR09")
@@
 		)
 		(instances
-			(project "macroboard-rev1"
+			(project "macropad-rev1"
 				(path "/e2f35591-d2a5-4370-be80-1eddbbb1c064"
 					(reference "#PWR012")
@@
 		)
 		(instances
-			(project "macroboard-rev1"
+			(project "macropad-rev1"
 				(path "/e2f35591-d2a5-4370-be80-1eddbbb1c064"
 					(reference "#PWR07")
@@
 		)
 		(instances
-			(project "macroboard-rev1"
+			(project "macropad-rev1"
 				(path "/e2f35591-d2a5-4370-be80-1eddbbb1c064"
 					(reference "R7")
@@
 		)
 		(instances
-			(project "macroboard-rev1"
+			(project "macropad-rev1"
 				(path "/e2f35591-d2a5-4370-be80-1eddbbb1c064"
 					(reference "#PWR08")
@@
 			)
 		)
-		(property "Footprint" "LiveWires:LW_CherrySwitch"
+		(property "Footprint" "LiveWires:LW_CherrySwitch_DrillMarks"
 			(at 199.39 130.81 0)
 			(effects
@@
 		)
 		(instances
-			(project "macroboard-rev1"
+			(project "macropad-rev1"
 				(path "/e2f35591-d2a5-4370-be80-1eddbbb1c064"
 					(reference "SW7")
@@
 		)
 		(instances
-			(project "macroboard-rev1"
+			(project "macropad-rev1"
 				(path "/e2f35591-d2a5-4370-be80-1eddbbb1c064"
 					(reference "R6")
@@
 		)
 		(instances
-			(project "macroboard-rev1"
+			(project "macropad-rev1"
 				(path "/e2f35591-d2a5-4370-be80-1eddbbb1c064"
 					(reference "#PWR011")
@@
 		)
 		(instances
-			(project "macroboard-rev1"
+			(project "macropad-rev1"
 				(path "/e2f35591-d2a5-4370-be80-1eddbbb1c064"
 					(reference "#PWR018")
@@
 			)
 		)
-		(property "Footprint" "LiveWires:LW_CherrySwitch"
+		(property "Footprint" "LiveWires:LW_CherrySwitch_DrillMarks"
 			(at 52.07 97.79 0)
 			(effects
@@
 		)
 		(instances
-			(project "macroboard-rev1"
+			(project "macropad-rev1"
 				(path "/e2f35591-d2a5-4370-be80-1eddbbb1c064"
 					(reference "SW4")
@@
 		)
 		(instances
-			(project "macroboard-rev1"
+			(project "macropad-rev1"
 				(path "/e2f35591-d2a5-4370-be80-1eddbbb1c064"
 					(reference "#PWR03")
@@
 		)
 		(instances
-			(project "macroboard-rev1"
+			(project "macropad-rev1"
 				(path "/e2f35591-d2a5-4370-be80-1eddbbb1c064"
 					(reference "#PWR01")
@@
 		)
 		(instances
-			(project "macroboard-rev1"
+			(project "macropad-rev1"
 				(path "/e2f35591-d2a5-4370-be80-1eddbbb1c064"
 					(reference "R4")
@@
 		)
 		(instances
-			(project "macroboard-rev1"
+			(project "macropad-rev1"
 				(path "/e2f35591-d2a5-4370-be80-1eddbbb1c064"
 					(reference "#PWR016")
@@
 			)
 		)
-		(property "Footprint" "LiveWires:LW_CherrySwitch"
+		(property "Footprint" "LiveWires:LW_CherrySwitch_DrillMarks"
 			(at 52.07 73.66 0)
 			(effects
@@
 		)
 		(instances
-			(project "macroboard-rev1"
+			(project "macropad-rev1"
 				(path "/e2f35591-d2a5-4370-be80-1eddbbb1c064"
 					(reference "SW1")
@@
 		)
 		(instances
-			(project "macroboard-rev1"
+			(project "macropad-rev1"
 				(path "/e2f35591-d2a5-4370-be80-1eddbbb1c064"
 					(reference "R2")
@@
 		)
 		(instances
-			(project "macroboard-rev1"
+			(project "macropad-rev1"
 				(path "/e2f35591-d2a5-4370-be80-1eddbbb1c064"
 					(reference "R1")
@@
 			)
 		)
-		(property "Footprint" "LiveWires:LW_CherrySwitch"
+		(property "Footprint" "LiveWires:LW_CherrySwitch_DrillMarks"
 			(at 199.39 123.19 0)
 			(effects
@@
 		)
 		(instances
-			(project "macroboard-rev1"
+			(project "macropad-rev1"
 				(path "/e2f35591-d2a5-4370-be80-1eddbbb1c064"
 					(reference "SW6")
@@
 		)
 		(instances
-			(project "macroboard-rev1"
+			(project "macropad-rev1"
 				(path "/e2f35591-d2a5-4370-be80-1eddbbb1c064"
 					(reference "U1")
@@
 		)
 		(instances
-			(project "macroboard-rev1"
+			(project "macropad-rev1"
 				(path "/e2f35591-d2a5-4370-be80-1eddbbb1c064"
 					(reference "SW10")
@@
 		)
 		(instances
-			(project "macroboard-rev1"
+			(project "macropad-rev1"
 				(path "/e2f35591-d2a5-4370-be80-1eddbbb1c064"
 					(reference "R3")
@@
 		)
 		(instances
-			(project "macroboard-rev1"
+			(project "macropad-rev1"
 				(path "/e2f35591-d2a5-4370-be80-1eddbbb1c064"
 					(reference "Q4")
@@
 		)
 		(instances
-			(project "macroboard-rev1"
+			(project "macropad-rev1"
 				(path "/e2f35591-d2a5-4370-be80-1eddbbb1c064"
 					(reference "#PWR013")
@@
 		)
 		(instances
-			(project "macroboard-rev1"
+			(project "macropad-rev1"
 				(path "/e2f35591-d2a5-4370-be80-1eddbbb1c064"
 					(reference "D3")
@@
 		)
 		(instances
-			(project "macroboard-rev1"
+			(project "macropad-rev1"
 				(path "/e2f35591-d2a5-4370-be80-1eddbbb1c064"
 					(reference "#PWR014")
@@
 		)
 		(instances
-			(project "macroboard-rev1"
+			(project "macropad-rev1"
 				(path "/e2f35591-d2a5-4370-be80-1eddbbb1c064"
 					(reference "R5")

Commit message: Working PCB
Parts:
- SW1, SW2, SW3, SW4, SW5, SW6, SW7, SW8, SW9: footprint LiveWires:LW_CherrySwitch_DrillMarks -> LiveWires:LW_CherrySwitch
Changed lines of the file:
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@@
 			)
 		)
-		(property "Footprint" "LiveWires:LW_CherrySwitch_DrillMarks"
+		(property "Footprint" "LiveWires:LW_CherrySwitch"
 			(at 52.07 62.23 0)
 			(effects
@@
 			)
 		)
-		(property "Footprint" "LiveWires:LW_CherrySwitch_DrillMarks"
+		(property "Footprint" "LiveWires:LW_CherrySwitch"
 			(at 199.39 115.57 0)
 			(effects
@@
 			)
 		)
-		(property "Footprint" "LiveWires:LW_CherrySwitch_DrillMarks"
+		(property "Footprint" "LiveWires:LW_CherrySwitch"
 			(at 52.07 90.17 0)
 			(effects
@@
 			)
 		)
-		(property "Footprint" "LiveWires:LW_CherrySwitch_DrillMarks"
+		(property "Footprint" "LiveWires:LW_CherrySwitch"
 			(at 52.07 82.55 0)
 			(effects
@@
 			)
 		)
-		(property "Footprint" "LiveWires:LW_CherrySwitch_DrillMarks"
+		(property "Footprint" "LiveWires:LW_CherrySwitch"
 			(at 199.39 138.43 0)
 			(effects
@@
 			)
 		)
-		(property "Footprint" "LiveWires:LW_CherrySwitch_DrillMarks"
+		(property "Footprint" "LiveWires:LW_CherrySwitch"
 			(at 199.39 130.81 0)
 			(effects
@@
 			)
 		)
-		(property "Footprint" "LiveWires:LW_CherrySwitch_DrillMarks"
+		(property "Footprint" "LiveWires:LW_CherrySwitch"
 			(at 52.07 97.79 0)
 			(effects
@@
 			)
 		)
-		(property "Footprint" "LiveWires:LW_CherrySwitch_DrillMarks"
+		(property "Footprint" "LiveWires:LW_CherrySwitch"
 			(at 52.07 73.66 0)
 			(effects
@@
 			)
 		)
-		(property "Footprint" "LiveWires:LW_CherrySwitch_DrillMarks"
+		(property "Footprint" "LiveWires:LW_CherrySwitch"
 			(at 199.39 123.19 0)
 			(effects
